Commit message: Imported upstream version '4.0.4' of 'upstream'

File: pmb2_description/urdf/wheels/wheel.ros2_control.xacro (robot description, xacro)
@@ -17,9 +17,9 @@
     </joint>
     <transmission name="wheel_${side}_trans">
-      <type>transmission_interface/SimpleTransmission</type>
-      <actuator name="wheel_${side}_motor">
+      <plugin>transmission_interface/SimpleTransmission</plugin>
+      <actuator name="wheel_${side}_motor" role="actuator1">
         <mechanicalReduction>1.0</mechanicalReduction>
       </actuator>
-      <joint name="wheel_${side}_joint">
+      <joint name="wheel_${side}_joint" role="joint1">
         <hardwareInterface>hardware_interface/VelocityJointInterface</hardwareInterface>
         <hardwareInterface>hardware_interface/JointStateInterface</hardwareInterface>
