Commit message: Imported upstream version '5.1.1' of 'upstream'

File: pmb2_description/urdf/wheels/caster.gazebo.xacro (robot description, xacro)
@@ -16,36 +16,16 @@
     <!-- Contact model for the caster wheel surface -->
     <gazebo reference="caster_${side}_1_link">
-      <kp>1000000.0</kp>
-      <kd>10000.0</kd>
-      <mu1>0.0</mu1>
-      <mu2>0.0</mu2>
-      <!--<fdir1>1 0 0</fdir1>-->
-      <max_vel>1.0</max_vel>
-      <min_depth>0.005</min_depth>
+      <mu1>0.1</mu1>
+      <mu2>0.1</mu2>
+      <kp>100000.0</kp>
+      <kd>1.0</kd>
       <material>Gazebo/DarkGrey</material>
     </gazebo>
     <gazebo reference="caster_${side}_2_link">
-      <kp>1000000.0</kp>
-      <kd>10000.0</kd>
-      <mu1>0.0</mu1>
-      <mu2>0.0</mu2>
-      <!--<fdir1>1 0 0</fdir1>-->
-      <max_vel>1.0</max_vel>
-      <min_depth>0.005</min_depth>
+      <mu1>0.1</mu1>
+      <mu2>0.1</mu2>
+      <kp>100000.0</kp>
+      <kd>1.0</kd>
       <material>Gazebo/DarkGrey</material>
-    </gazebo>
-    <gazebo reference="caster_{side}_1_joint">
-      <physics>
-        <ode>
-          <implicit_spring_damper>0</implicit_spring_damper>
-        </ode>
-      </physics>
-    </gazebo>
-    <gazebo reference="caster_{side}_2_joint">
-      <physics>
-        <ode>
-          <implicit_spring_damper>0</implicit_spring_damper>
-        </ode>
-      </physics>
     </gazebo>
   </xacro:macro>

File: pmb2_description/urdf/wheels/wheel.gazebo.xacro (robot description, xacro)
@@ -16,23 +16,11 @@
     <!-- Contact model for the wheel surface -->
     <gazebo reference="wheel_${side}_link">
+      <mu1>1.0</mu1>
+      <mu2>1.0</mu2>
       <kp>1000000.0</kp>
       <kd>100.0</kd>
-      <friction>
-        <ode>
-          <mu>1.0</mu>
-          <mu2>1.0</mu2>
-        </ode>
-      </friction>
-      <!--<fdir1>1 0 0</fdir1>-->
-      <max_vel>1.0</max_vel>
-      <min_depth>0.002</min_depth>
+      <minDepth>0.002</minDepth>
+      <maxVel>1.0</maxVel>
       <material>Gazebo/DarkGrey</material>
-    </gazebo>
-    <gazebo reference="wheel_{side}_joint">
-      <physics>
-        <ode>
-          <implicit_spring_damper>1</implicit_spring_damper>
-        </ode>
-      </physics>
     </gazebo>
   </xacro:macro>

File: pmb2_description/urdf/wheels/wheel.urdf.xacro (robot description, xacro)
@@ -31,6 +31,5 @@
         <origin xyz="0 0 0" rpy="0 0 0"/>
         <geometry>
-          <sphere radius="${radius}" />
-          <!-- length="${width}"/> -->
+          <cylinder radius="${radius}" length="${width}"/>
         </geometry>
       </collision>
