Commit message: Rebase from 'upstream'

File: pmb2_description/robots/pmb2.urdf.xacro (robot description, xacro)
@@ -14,5 +14,5 @@
 <robot  xmlns:xacro="http://ros.org/wiki/xacro"
         name="pmb2" >
-  <xacro:arg name="use_sim" default="true"/>
+  <xacro:arg name="use_sim" default="false"/>
   <xacro:arg name="laser_model" default="sick-571"/> <!-- no-laser, hokuyo, sick-551, sick-561, sick-571-->
   <xacro:arg name="courier_rgbd_sensors" default="false"/> <!-- false, true-->

File: pmb2_description/ros2_control/ros2_control.urdf.xacro (robot description, xacro)
@@ -14,5 +14,5 @@
 <robot xmlns:xacro="http://ros.org/wiki/xacro"
        name="pmb2" >
-<xacro:macro name="pmb2_ros2_control" params="use_sim:=^|true">
+<xacro:macro name="pmb2_ros2_control" params="use_sim:=^|false">
     <xacro:include filename="$(find pmb2_description)/urdf/wheels/wheel.ros2_control.xacro"/>
     <xacro:include filename="$(find pmb2_description)/urdf/sensors/sensors.ros2_control.xacro"/>

File: pmb2_description/urdf/sensors/hokuyo_urg_04lx_ug01_laser.gazebo.xacro (robot description, xacro)
@@ -40,5 +40,5 @@
           </noise>
         </ray>
-      	<plugin name="bytes_laserscan" filename="libgazebo_ros_ray_sensor.so">
+      	<plugin name="${name}" filename="libgazebo_ros_ray_sensor.so">
           <ros>
       	    <remapping>~/out:=${ros_topic}</remapping>

File: pmb2_description/urdf/sensors/sick_tim551_laser.gazebo.xacro (robot description, xacro)
@@ -40,5 +40,5 @@
           </noise>
         </ray>
-      	<plugin name="bytes_laserscan" filename="libgazebo_ros_ray_sensor.so">
+      	<plugin name="${name}" filename="libgazebo_ros_ray_sensor.so">
           <ros>
       	    <remapping>~/out:=${ros_topic}</remapping>

File: pmb2_description/urdf/sensors/sick_tim561_laser.gazebo.xacro (robot description, xacro)
@@ -40,5 +40,5 @@
           </noise>
         </ray>
-      	<plugin name="bytes_laserscan" filename="libgazebo_ros_ray_sensor.so">
+      	<plugin name="${name}" filename="libgazebo_ros_ray_sensor.so">
           <ros>
       	    <remapping>~/out:=${ros_topic}</remapping>

File: pmb2_description/urdf/sensors/sick_tim571_laser.gazebo.xacro (robot description, xacro)
@@ -40,5 +40,5 @@
           </noise>
         </ray>
-      	<plugin name="bytes_laserscan" filename="libgazebo_ros_ray_sensor.so">
+      	<plugin name="${name}" filename="libgazebo_ros_ray_sensor.so">
           <ros>
       	    <remapping>~/out:=${ros_topic}</remapping>
