Commit message: Imported upstream version '4.0.5' of 'upstream'

File: pmb2_description/urdf/sensors/imu.urdf.xacro (robot description, xacro)
@@ -1,10 +1,15 @@
 <?xml version="1.0"?>
 <!--
-  Copyright (c) 2011-2012, PAL Robotics, S.L.
-  All rights reserved.
-  This work is licensed under the Creative Commons Attribution-NonCommercial-NoDerivs 3.0 Unported License.
-  To view a copy of this license, visit http://creativecommons.org/licenses/by-nc-nd/3.0/ or send a letter to
-  Creative Commons, 444 Castro Street, Suite 900, Mountain View, California, 94041, USA.
--->
+  Copyright (c) 2022 PAL Robotics S.L. All rights reserved.
+  Licensed under the Apache License, Version 2.0 (the "License");
+  you may not use this file except in compliance with the License.
+  You may obtain a copy of the License at
+      http://www.apache.org/licenses/LICENSE-2.0
+  Unless required by applicable law or agreed to in writing, software
+  distributed under the License is distributed on an "AS IS" BASIS,
+  WITHOUT WARRANTIES OR CONDITIONS OF ANY KIND, either express or implied.
+  See the License for the specific language governing permissions and
+  limitations under the License.
+ -->
 <robot xmlns:xacro="http://ros.org/wiki/xacro">
   <xacro:macro name="imu_sensor" params="name parent *origin update_rate">

File: pmb2_description/urdf/sensors/microphone.urdf.xacro (robot description, xacro)
@@ -1,10 +1,15 @@
 <?xml version="1.0"?>
 <!--
-  Copyright (c) 2013, PAL Robotics, S.L.
-  All rights reserved.
-  This work is licensed under the Creative Commons Attribution-NonCommercial-NoDerivs 3.0 Unported License.
-  To view a copy of this license, visit http://creativecommons.org/licenses/by-nc-nd/3.0/ or send a letter to
-  Creative Commons, 444 Castro Street, Suite 900, Mountain View, California, 94041, USA.
--->
+  Copyright (c) 2022 PAL Robotics S.L. All rights reserved.
+  Licensed under the Apache License, Version 2.0 (the "License");
+  you may not use this file except in compliance with the License.
+  You may obtain a copy of the License at
+      http://www.apache.org/licenses/LICENSE-2.0
+  Unless required by applicable law or agreed to in writing, software
+  distributed under the License is distributed on an "AS IS" BASIS,
+  WITHOUT WARRANTIES OR CONDITIONS OF ANY KIND, either express or implied.
+  See the License for the specific language governing permissions and
+  limitations under the License.
+ -->
 <robot xmlns:xacro="http://ros.org/wiki/xacro">
   <!-- Macro -->

File: pmb2_description/urdf/sensors/range.gazebo.xacro (robot description, xacro)
@@ -1,10 +1,15 @@
 <?xml version="1.0"?>
 <!--
-  Copyright (c) 2011, PAL Robotics, S.L.
-  All rights reserved.
-  This work is licensed under the Creative Commons Attribution-NonCommercial-NoDerivs 3.0 Unported License.
-  To view a copy of this license, visit http://creativecommons.org/licenses/by-nc-nd/3.0/ or send a letter to
-  Creative Commons, 444 Castro Street, Suite 900, Mountain View, California, 94041, USA.
--->
+  Copyright (c) 2022 PAL Robotics S.L. All rights reserved.
+  Licensed under the Apache License, Version 2.0 (the "License");
+  you may not use this file except in compliance with the License.
+  You may obtain a copy of the License at
+      http://www.apache.org/licenses/LICENSE-2.0
+  Unless required by applicable law or agreed to in writing, software
+  distributed under the License is distributed on an "AS IS" BASIS,
+  WITHOUT WARRANTIES OR CONDITIONS OF ANY KIND, either express or implied.
+  See the License for the specific language governing permissions and
+  limitations under the License.
+ -->
 <robot xmlns:xacro="http://ros.org/wiki/xacro">
   <xacro:macro name="range_gazebo" params="name ros_topic update_rate maxRange minRange fov radiation" >

File: pmb2_description/urdf/sensors/range.urdf.xacro (robot description, xacro)
@@ -1,10 +1,15 @@
 <?xml version="1.0"?>
 <!--
-  Copyright (c) 2011, PAL Robotics, S.L.
-  All rights reserved.
-  This work is licensed under the Creative Commons Attribution-NonCommercial-NoDerivs 3.0 Unported License.
-  To view a copy of this license, visit http://creativecommons.org/licenses/by-nc-nd/3.0/ or send a letter to
-  Creative Commons, 444 Castro Street, Suite 900, Mountain View, California, 94041, USA.
--->
+  Copyright (c) 2022 PAL Robotics S.L. All rights reserved.
+  Licensed under the Apache License, Version 2.0 (the "License");
+  you may not use this file except in compliance with the License.
+  You may obtain a copy of the License at
+      http://www.apache.org/licenses/LICENSE-2.0
+  Unless required by applicable law or agreed to in writing, software
+  distributed under the License is distributed on an "AS IS" BASIS,
+  WITHOUT WARRANTIES OR CONDITIONS OF ANY KIND, either express or implied.
+  See the License for the specific language governing permissions and
+  limitations under the License.
+ -->
 <robot xmlns:xacro="http://ros.org/wiki/xacro">
   <xacro:include filename="$(find pmb2_description)/urdf/sensors/range.gazebo.xacro" />

Commit message: Imported upstream version '5.0.20' of 'upstream'

File: pmb2_description/gazebo/gazebo.urdf.xacro (robot description, xacro)
@@ -13,8 +13,7 @@
  -->
 <robot xmlns:sensor="http://playerstage.sourceforge.net/gazebo/xmlschema/#sensor"
-       xmlns:controller="http://playerstage.sourceforge.net/gazebo/xmlschema/#controller"
-       xmlns:interface="http://playerstage.sourceforge.net/gazebo/xmlschema/#interface"
-       xmlns:xacro="http://ros.org/wiki/xacro"
-       name="pmb2">
+  xmlns:controller="http://playerstage.sourceforge.net/gazebo/xmlschema/#controller"
+  xmlns:interface="http://playerstage.sourceforge.net/gazebo/xmlschema/#interface"
+  xmlns:xacro="http://ros.org/wiki/xacro" name="pmb2">
   <gazebo>
     <plugin filename="libgazebo_ros2_control.so" name="gazebo_ros2_control">
@@ -34,30 +33,7 @@
       <update_rate>100.0</update_rate>
       <xacro:if value="${is_multiple}">
-          <namespace>/${nsp}</namespace>
+        <namespace>/${nsp}</namespace>
       </xacro:if>
     </plugin>
-  </gazebo>
-  <gazebo reference="base_imu_link">
-    <sensor name="imu_sensor" type="imu">
-      <always_on>1</always_on>
-      <update_rate>10.0</update_rate>
-      <imu>
-        <noise>
-          <type>gaussian</type>
-          <rate>
-            <mean>0.0</mean>
-            <stddev>2e-4</stddev>
-            <bias_mean>0.0000075</bias_mean>
-            <bias_stddev>0.0000008</bias_stddev>
-          </rate>
-          <accel>
-            <mean>0.0</mean>
-            <stddev>1.7e-2</stddev>
-            <bias_mean>0.1</bias_mean>
-            <bias_stddev>0.001</bias_stddev>
-          </accel>
-        </noise>
-      </imu>
-    </sensor>
   </gazebo>
   <!-- define global properties -->

File: pmb2_description/urdf/base/base.urdf.xacro (robot description, xacro)
@@ -20,17 +20,17 @@
   <xacro:include filename="$(find pmb2_description)/urdf/objects/antenna.urdf.xacro"/>
   <!-- Wheel characteristics -->
-  <xacro:property name="wheel_radius"     value="0.0985"/>
-  <xacro:property name="wheel_width"      value="0.040"/>
+  <xacro:property name="wheel_radius" value="0.0985"/>
+  <xacro:property name="wheel_width" value="0.040"/>
   <xacro:property name="wheel_separation" value="0.4044"/>
-  <xacro:property name="wheel_torque"     value="6.0"/>
-  <xacro:property name="wheel_velocity"   value="1.0"/>
+  <xacro:property name="wheel_torque" value="6.0"/>
+  <xacro:property name="wheel_velocity" value="1.0"/>
   <!-- Caster wheel characteristics -->
-  <xacro:property name="caster_radius"       value="0.025"/>
-  <xacro:property name="caster_width"        value="0.015"/>
+  <xacro:property name="caster_radius" value="0.025"/>
+  <xacro:property name="caster_width" value="0.015"/>
   <xacro:property name="caster_separation_x" value="0.343"/>
   <xacro:property name="caster_separation_y" value="0.204"/>
-  <xacro:property name="caster_offset_x"     value="-0.002"/>
-  <xacro:property name="caster_offset_y"     value="0.0"/>
-  <xacro:property name="caster_offset_z"     value="-0.0335"/>
+  <xacro:property name="caster_offset_x" value="-0.002"/>
+  <xacro:property name="caster_offset_y" value="0.0"/>
+  <xacro:property name="caster_offset_z" value="-0.0335"/>
   <xacro:macro name="base" params="name">
     <!-- Base -->
@@ -39,7 +39,5 @@
         <origin xyz="-0.00000106 0.00000109 0.0000387" rpy="0 0 0"/>
         <mass value="28.26649"/>
-        <inertia ixx="0.465408937" ixy="0.002160024" ixz="-0.001760255"
-                 iyy="0.483193291" iyz="-0.000655952"
-                 izz="0.550939703"/>
+        <inertia ixx="0.465408937" ixy="0.002160024" ixz="-0.001760255" iyy="0.483193291" iyz="-0.000655952" izz="0.550939703"/>
       </inertial>
       <visual>
@@ -68,5 +66,5 @@
       <parent link="${name}_footprint"/>
     </joint>
-  <!-- gazebo parameters are given here for base_link thru base_footprint -->
+    <!-- gazebo parameters are given here for base_link thru base_footprint -->
     <gazebo reference="${name}_footprint">
       <kp>100000000.0</kp>
@@ -93,10 +91,10 @@
     <!-- Wheels -->
     <xacro:wheel side="right" reflect=" 1.0" radius="${wheel_radius}" width="${wheel_width}" torque="${wheel_torque}" velocity="${wheel_velocity}" separation="${wheel_separation}" parent="${name}"/>
-    <xacro:wheel side="left"  reflect="-1.0" radius="${wheel_radius}" width="${wheel_width}" torque="${wheel_torque}" velocity="${wheel_velocity}" separation="${wheel_separation}" parent="${name}"/>
+    <xacro:wheel side="left" reflect="-1.0" radius="${wheel_radius}" width="${wheel_width}" torque="${wheel_torque}" velocity="${wheel_velocity}" separation="${wheel_separation}" parent="${name}"/>
     <!-- Casters wheels -->
     <xacro:caster side="front_right" radius="${caster_radius}" width="${caster_width}" separation_x="${ caster_separation_x}" separation_y="${ caster_separation_y}" offset_x="${caster_offset_x}" offset_y="${caster_offset_y}" offset_z="${caster_offset_z}" parent="${name}"/>
-    <xacro:caster side="front_left"  radius="${caster_radius}" width="${caster_width}" separation_x="${ caster_separation_x}" separation_y="${-caster_separation_y}" offset_x="${caster_offset_x}" offset_y="${caster_offset_y}" offset_z="${caster_offset_z}" parent="${name}"/>
-    <xacro:caster side="back_right"  radius="${caster_radius}" width="${caster_width}" separation_x="${-caster_separation_x}" separation_y="${ caster_separation_y}" offset_x="${caster_offset_x}" offset_y="${caster_offset_y}" offset_z="${caster_offset_z}" parent="${name}"/>
-    <xacro:caster side="back_left"   radius="${caster_radius}" width="${caster_width}" separation_x="${-caster_separation_x}" separation_y="${-caster_separation_y}" offset_x="${caster_offset_x}" offset_y="${caster_offset_y}" offset_z="${caster_offset_z}" parent="${name}"/>
+    <xacro:caster side="front_left" radius="${caster_radius}" width="${caster_width}" separation_x="${ caster_separation_x}" separation_y="${-caster_separation_y}" offset_x="${caster_offset_x}" offset_y="${caster_offset_y}" offset_z="${caster_offset_z}" parent="${name}"/>
+    <xacro:caster side="back_right" radius="${caster_radius}" width="${caster_width}" separation_x="${-caster_separation_x}" separation_y="${ caster_separation_y}" offset_x="${caster_offset_x}" offset_y="${caster_offset_y}" offset_z="${caster_offset_z}" parent="${name}"/>
+    <xacro:caster side="back_left" radius="${caster_radius}" width="${caster_width}" separation_x="${-caster_separation_x}" separation_y="${-caster_separation_y}" offset_x="${caster_offset_x}" offset_y="${caster_offset_y}" offset_z="${caster_offset_z}" parent="${name}"/>
   </xacro:macro>
 </robot>

File: pmb2_description/urdf/base/base_sensors.urdf.xacro (robot description, xacro)
@@ -1,5 +1,5 @@
 <?xml version="1.0"?>
 <!--
-  Copyright (c) 2022 PAL Robotics S.L. All rights reserved.
+  Copyright (c) 2024 PAL Robotics S.L. All rights reserved.
   Licensed under the Apache License, Version 2.0 (the "License");
   you may not use this file except in compliance with the License.
@@ -13,4 +13,9 @@
  -->
 <robot xmlns:xacro="http://ros.org/wiki/xacro">
+  <!-- PROPERTIES -->
+  <xacro:property name="base_laser_x" value="0.202"/>
+  <xacro:property name="base_laser_y" value="0.0"/>
+  <xacro:property name="base_laser_z" value="-0.004"/>
+  <!-- INCLUDES -->
   <xacro:include filename="$(find pmb2_description)/urdf/base/base.urdf.xacro"/>
   <xacro:include filename="$(find pmb2_description)/urdf/sensors/hokuyo_urg_04lx_ug01_laser.urdf.xacro"/>
@@ -20,14 +25,10 @@
   <xacro:include filename="$(find pmb2_description)/urdf/sensors/range.urdf.xacro"/>
   <xacro:include filename="$(find pmb2_description)/urdf/sensors/microphone.urdf.xacro"/>
-  <!-- Laser characteristics -->
-  <xacro:property name="base_laser_x" value="0.202"/>
-  <xacro:property name="base_laser_y" value="0.0"/>
-  <xacro:property name="base_laser_z" value="-0.004"/>
-  <!-- laser_model can be: false, hokuyo, sick-551, sick-561, sick-571-->
+  <!-- MACRO DEFINITION -->
   <xacro:macro name="base_sensors" params=" name laser_model:=sick-571 sonars:=false microphone:=false ">
     <xacro:if value="${laser_model == 'hokuyo'}">
       <!-- Laser -->
       <!-- Theoretic FOV = 220 -->
-      <xacro:hokuyo_urg_04lx_ug01_laser name="${name}_laser" parent="${name}" ros_topic="scan_raw" update_rate="10" min_angle="${-110 * deg_to_rad}" max_angle="${110 * deg_to_rad}" >
+      <xacro:hokuyo_urg_04lx_ug01_laser name="${name}_laser" parent="${name}" ros_topic="scan_raw" update_rate="10" min_angle="${-110 * deg_to_rad}" max_angle="${110 * deg_to_rad}">
         <origin xyz="${base_laser_x} ${base_laser_y} ${base_laser_z}" rpy="0 0 0" />
       </xacro:hokuyo_urg_04lx_ug01_laser>
@@ -36,5 +37,5 @@
       <!-- Laser -->
       <!-- Theoretic FOV = 220 -->
-      <xacro:sick_tim551_laser name="${name}_laser" parent="${name}" ros_topic="scan_raw" update_rate="10" min_angle="${-110 * deg_to_rad}" max_angle="${110 * deg_to_rad}" >
+      <xacro:sick_tim551_laser name="${name}_laser" parent="${name}" ros_topic="scan_raw" update_rate="10" min_angle="${-110 * deg_to_rad}" max_angle="${110 * deg_to_rad}">
         <origin xyz="${base_laser_x} ${base_laser_y} ${base_laser_z}" rpy="0 0 0" />
       </xacro:sick_tim551_laser>
@@ -43,5 +44,5 @@
       <!-- Laser -->
       <!-- Theoretic FOV = 220 -->
-      <xacro:sick_tim561_laser name="${name}_laser" parent="${name}" ros_topic="scan_raw" update_rate="10" min_angle="${-110 * deg_to_rad}" max_angle="${110 * deg_to_rad}" >
+      <xacro:sick_tim561_laser name="${name}_laser" parent="${name}" ros_topic="scan_raw" update_rate="10" min_angle="${-110 * deg_to_rad}" max_angle="${110 * deg_to_rad}">
         <origin xyz="${base_laser_x} ${base_laser_y} ${base_laser_z}" rpy="0 0 0" />
       </xacro:sick_tim561_laser>
@@ -50,5 +51,5 @@
       <!-- Laser -->
       <!-- Theoretic FOV = 220 -->
-      <xacro:sick_tim571_laser name="${name}_laser" parent="${name}" ros_topic="scan_raw" update_rate="10" min_angle="${-110 * deg_to_rad}" max_angle="${110 * deg_to_rad}" >
+      <xacro:sick_tim571_laser name="${name}_laser" parent="${name}" ros_topic="scan_raw" update_rate="10" min_angle="${-110 * deg_to_rad}" max_angle="${110 * deg_to_rad}">
         <origin xyz="${base_laser_x} ${base_laser_y} ${base_laser_z}" rpy="0 0 0" />
       </xacro:sick_tim571_laser>

File: pmb2_description/urdf/sensors/imu.urdf.xacro (robot description, xacro)
@@ -1,5 +1,5 @@
 <?xml version="1.0"?>
 <!--
-  Copyright (c) 2022 PAL Robotics S.L. All rights reserved.
+  Copyright (c) 2024 PAL Robotics S.L. All rights reserved.
   Licensed under the Apache License, Version 2.0 (the "License");
   you may not use this file except in compliance with the License.
@@ -13,4 +13,7 @@
  -->
 <robot xmlns:xacro="http://ros.org/wiki/xacro">
+  <!-- INCLUDES -->
+  <xacro:include filename="$(find pmb2_description)/urdf/sensors/imu.gazebo.xacro" />
+  <!-- MACRO DEFINITION -->
   <xacro:macro name="imu_sensor" params="name parent *origin update_rate">
     <link name="${name}_link">
@@ -32,27 +35,6 @@
       <xacro:insert_block name="origin"/>
     </joint>
-    <gazebo reference="${name}_link">
-      <sensor name="${name}_sensor" type="imu">
-        <always_on>1</always_on>
-        <update_rate>100.0</update_rate>
-        <imu>
-          <noise>
-            <type>gaussian</type>
-            <rate>
-              <mean>0.0</mean>
-              <stddev>2e-4</stddev>
-              <bias_mean>0.0000075</bias_mean>
-              <bias_stddev>0.0000008</bias_stddev>
-            </rate>
-            <accel>
-              <mean>0.0</mean>
-              <stddev>1.7e-2</stddev>
-              <bias_mean>0.1</bias_mean>
-              <bias_stddev>0.001</bias_stddev>
-            </accel>
-          </noise>
-        </imu>
-      </sensor>
-    </gazebo>
+    <!-- Gazebo config-->
+    <xacro:imu_gazebo name="${name}" update_rate="${update_rate}" />
   </xacro:macro>
 </robot>

File: pmb2_description/urdf/sensors/sick_tim551_laser.gazebo.xacro (robot description, xacro)
@@ -37,5 +37,5 @@
             <type>gaussian</type>
             <mean>0.0</mean>
-            <stddev>0.06</stddev>
+            <stddev>0.01</stddev>
           </noise>
         </ray>

File: pmb2_description/urdf/sensors/sick_tim561_laser.gazebo.xacro (robot description, xacro)
@@ -37,5 +37,5 @@
             <type>gaussian</type>
             <mean>0.0</mean>
-            <stddev>0.06</stddev>
+            <stddev>0.01</stddev>
           </noise>
         </ray>

File: pmb2_description/urdf/sensors/sick_tim571_laser.gazebo.xacro (robot description, xacro)
@@ -37,5 +37,5 @@
             <type>gaussian</type>
             <mean>0.0</mean>
-            <stddev>0.06</stddev>
+            <stddev>0.01</stddev>
           </noise>
         </ray>
